File: board/xmas_orn/xmas_orn.kicad_sch (KiCad schematic)
At the start: 17 parts, among them J1 Conn_01x07_Socket, J3 USB_C_Receptacle_USB2.0_16P, SW1 RST, SW2 BOOT, U1 ESP32-S3-MINI-1, U2 TLV75733PDBV

Commit message: Add xmas_hub 12 V -> 4 x 5 V power hub board; ornament rev 2 (WROOM-1, barrel jack)
board/xmas_hub (new KiCad 10 project): the base-of-tree distribution board for
the star topology. A 12 V barrel supply (DC-005, 5 A PTC, SMAJ15A TVS, AOD417
P-FET reverse-polarity protection, 100 uF bulk) feeds four independent
TPS54302 synchronous bucks, each with its own 2.6 A PTC, LED and 5.08 mm screw
terminal, so a fault on one arm leaves the other three running. Arms are set to
4.95 V (100k/13.7k) and feed the ornaments' DC-002 jacks over 20-22 AWG twin
lead. 80 x 66 mm, two layers, ground pours both sides.

- Schematic and PCB were bootstrapped by scripts/gen_sch.py and gen_pcb.py
  (KiCad symbol libs + bundled pcbnew); ERC and DRC with schematic parity pass.
- Every BOM line carries a verified "LCSC Part #" field; JLCPCB gerbers, drill,
  position and BOM files are in production/.
- Project footprint for the DC-005 jack: its sleeve is the lateral pin and the
  switch contact is in line with the centre pin, the opposite of KiCad's generic
  BarrelJack_Horizontal, which would have put GND on the contact that opens when
  a plug is inserted.
- docs/ has schematic/top/bottom PDFs and the datasheets the design was checked
  against; README documents the design, BOM, cable guidance and regeneration.

board/xmas_orn rev 2: ESP32-S3-WROOM-1-N16R8 module replaces the MINI-1-N8,
board grows to 27.5 x 41.5 mm, USB-C VBUS and a DNP DC-002 5 V barrel jack are
Schottky OR-ed into VIN. Project footprint/3D model for the DC-002 jack, rev 2
docs and JLCPCB outputs, and sdkconfig.rev2.defaults as an overlay for the
16 MB flash / 8 MB octal PSRAM module. Top-level README gains the rev 2 notes
and a pointer to the hub; .gitignore covers KiCad backups and lock files.

Co-Authored-By: Claude Fable 5.1 <noreply@anthropic.com>
Parts:
- added D3, D4: B5819W, Diode_SMD:D_SOD-123, symbol Device:D_Schottky
- added J2: DC-002, xmas_orn:DC-002_BarrelJack_3.5x1.3mm_Horizontal, symbol Connector:Barrel_Jack_Switch
- U1: value ESP32-S3-MINI-1 -> ESP32-S3-WROOM-1; footprint RF_Module:ESP32-S2-MINI-1 -> RF_Module:ESP32-S3-WROOM-1; symbol RF_Module:ESP32-S3-MINI-1 -> RF_Module:ESP32-S3-WROOM-1; LCSC Part # (none) -> C2913202; MPN ESP32-S3-MINI-1-N8 -> ESP32-S3-WROOM-1-N16R8
Connections:
- net EN: now also U1.3 (EN); no longer U1.45 (EN)
- net GND: now also U1.40 (GND), U1.41 (GND), J2.2; no longer U1.2 (GND), U1.42 (GND), U1.43 (GND), U1.46 (GND), U1.47 (GND), U1.48 (GND), U1.49 (GND), U1.50 (GND), U1.51 (GND), U1.52 (GND), U1.53 (GND), U1.54 (GND), U1.55 (GND), U1.56 (GND), U1.57 (GND), U1.58 (GND), U1.59 (GND), U1.60 (GND), U1.61 (GND), U1.62 (GND), U1.63 (GND), U1.64 (GND), U1.65 (GND)
- net GPIO0: now also U1.27 (IO0); no longer U1.4 (IO0)
- net GPIO4: now also U1.4 (IO4); no longer U1.8 (IO4)
- net LCD_BLK: now also U1.7 (IO7); no longer U1.11 (IO7)
- net LCD_CS: now also U1.18 (IO10); no longer U1.14 (IO10)
- net LCD_DC: now also U1.17 (IO9); no longer U1.13 (IO9)
- net LCD_MOSI: now also U1.19 (IO11); no longer U1.15 (IO11)
- net LCD_SCLK: now also U1.20 (IO12); no longer U1.16 (IO12)
- net USB+: now also U1.14 (USB_D+); no longer U1.24 (USB_D+)
- net USB-: now also U1.13 (USB_D-); no longer U1.23 (USB_D-)
- net VCC: now also U1.2 (3V3); no longer U1.3 (3V3)
- net VIN: now also D3.1 (K), D4.1 (K); no longer J3.A4 (VBUS), J3.A9 (VBUS), J3.B4 (VBUS), J3.B9 (VBUS)
- new net VBUS: D3.2 (A), J3.A4 (VBUS), J3.A9 (VBUS), J3.B4 (VBUS), J3.B9 (VBUS)
- new net VJACK: D4.2 (A), J2.1
- no-connect marks 0 -> 1
Other:
- note added: "Power input OR-ing: USB VBUS (via D3) and the DC jack J2 (via D4) both feed VIN through Schottky diodes, so neither supply can back-feed the other when both are plugged in. Jack input must be 5 V DC (U2 max input 5.5 V). J2 is not populated by default."
- title: (none) -> xmas_orn
