File: board/xmas_hub/xmas_hub.kicad_pcb (KiCad board)
At the start: 2 copper layers, 80 x 66 mm, 66 parts, among them J1 DC-005 5.5x2.1mm, J2 ARM 1 5V, J3 ARM 2 5V, J4 ARM 3 5V, J5 ARM 4 5V, Q1 AOD417, U1 TPS54302DDCR, U2 TPS54302DDCR, U3 TPS54302DDCR, U4 TPS54302DDCR

Commit message: xmas_hub: size power copper for the 3 A arms and 5 A input
Audited every net with IPC-2221 (1 oz, 10 C rise). Input path jack -> PTC ->
TVS -> P-FET -> bus goes from 2.5 to 3.0 mm to match the 5 A PTC; the per-arm
12 V feed from 0.9 to 1.2 mm with a 0.6 mm stub into the VIN pin; the buck IC
ground pin, which returns ~1.8 A average at 3 A out, now lands on two
0.8/0.4 mm vias instead of one 0.6/0.3; the input-cap ground gets two 0.8/0.4
vias and the output-cap grounds one each. DRC with schematic parity still
passes. README gains a width/current table; production files and renders are
regenerated.

Co-Authored-By: Claude Fable 5.1 <noreply@anthropic.com>
Routing:
- net GND: track 47.0 -> 55.2 mm, vias 49 -> 57
- net +12V: track 109.3 -> 109.9 mm

Commit message: Gerbers: 0.05 mm solder-mask expansion on both boards
JLCPCB's minimum; at KiCad's default of 0 the mask opening equals the
pad and their DFM queried the identical USB-C shell slots on a sibling
order. pad_to_mask_clearance 0.05 in both boards, drill marks off,
gerber zips regenerated with the same file layout as before.

Co-Authored-By: Claude Fable 5.1 <noreply@anthropic.com>
Other:
- rule pad_to_mask_clearance: 0 -> 0.05
Changed lines of the file:
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@@
 	)
 	(setup
-		(pad_to_mask_clearance 0)
+		(pad_to_mask_clearance 0.05)
 		(allow_soldermask_bridges_in_footprints no)
 		(tenting
@@
 			(outputformat 1)
 			(mirror no)
-			(drillshape 1)
+			(drillshape 0)
 			(scaleselection 1)
 			(outputdirectory "")
